File: cables.kicad_sch (KiCad schematic)
At the start: 6 parts, among them J4 IDC20F, J5 DSUB19F, J5 DSUB19M, J7 DB25M

Commit message: readd second floppy connector
reference number changes
Parts:
- renumbered J5 to J6
Changed lines of the file:
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@@
         )
         (path "/c5fa29fb-f00a-43d2-879f-1e361b003a2a/4d4100c6-4979-4191-9309-82d4f93e23eb"
-          (reference "J3") (unit 1)
+          (reference "J4") (unit 1)
         )
       )
@@
         )
         (path "/c5fa29fb-f00a-43d2-879f-1e361b003a2a/4d4100c6-4979-4191-9309-82d4f93e23eb"
+          (reference "J7") (unit 1)
+        )
+      )
+    )
+  )
+  (symbol (lib_id "MyConnector:DSUB19_Male") (at 99.06 58.42 180) (unit 1)
+    (in_bom yes) (on_board no) (dnp no) (fields_autoplaced)
+    (property "Reference" "J6" (at 99.06 27.94 0)
+      (effects (font (size 1.27 1.27)))
+    )
+    (property "Value" "DSUB19M" (at 99.06 30.48 0)
+      (effects (font (size 1.27 1.27)))
+    )
+    (property "Footprint" "" (at 99.06 66.04 0)
+      (effects (font (size 1.27 1.27)) hide)
+    )
+    (property "Datasheet" " ~" (at 99.06 58.42 0)
+      (effects (font (size 1.27 1.27)) hide)
+    )
+    (pin "1")
+    (pin "10")
+    (pin "11")
+    (pin "12")
+    (pin "13")
+    (pin "14")
+    (pin "15")
+    (pin "16")
+    (pin "17")
+    (pin "18")
+    (pin "19")
+    (pin "2")
+    (pin "3")
+    (pin "4")
+    (pin "5")
+    (pin "6")
+    (pin "7")
+    (pin "8")
+    (pin "9")
+    (instances
+      (project "SmartDiskII"
+        (path "/c5fa29fb-f00a-43d2-879f-1e361b003a2a/4d4100c6-4979-4191-9309-82d4f93e23eb"
           (reference "J6") (unit 1)
-        )
-      )
-    )
-  )
-  (symbol (lib_id "MyConnector:DSUB19_Male") (at 99.06 58.42 180) (unit 1)
-    (in_bom yes) (on_board no) (dnp no) (fields_autoplaced)
-    (property "Reference" "J5" (at 99.06 27.94 0)
-      (effects (font (size 1.27 1.27)))
-    )
-    (property "Value" "DSUB19M" (at 99.06 30.48 0)
-      (effects (font (size 1.27 1.27)))
-    )
-    (property "Footprint" "" (at 99.06 66.04 0)
-      (effects (font (size 1.27 1.27)) hide)
-    )
-    (property "Datasheet" " ~" (at 99.06 58.42 0)
-      (effects (font (size 1.27 1.27)) hide)
-    )
-    (pin "1")
-    (pin "10")
-    (pin "11")
-    (pin "12")
-    (pin "13")
-    (pin "14")
-    (pin "15")
-    (pin "16")
-    (pin "17")
-    (pin "18")
-    (pin "19")
-    (pin "2")
-    (pin "3")
-    (pin "4")
-    (pin "5")
-    (pin "6")
-    (pin "7")
-    (pin "8")
-    (pin "9")
-    (instances
-      (project "SmartDiskII"
-        (path "/c5fa29fb-f00a-43d2-879f-1e361b003a2a/4d4100c6-4979-4191-9309-82d4f93e23eb"
-          (reference "J5") (unit 1)
         )
       )
@@
         )
         (path "/c5fa29fb-f00a-43d2-879f-1e361b003a2a/4d4100c6-4979-4191-9309-82d4f93e23eb"
-          (reference "J4") (unit 1)
+          (reference "J5") (unit 1)
         )
       )
@@
         )
         (path "/c5fa29fb-f00a-43d2-879f-1e361b003a2a/4d4100c6-4979-4191-9309-82d4f93e23eb"
+          (reference "J9") (unit 1)
+        )
+      )
+    )
+  )
+  (symbol (lib_id "Connector_Generic:Conn_01x20") (at 30.48 142.24 0) (mirror y) (unit 1)
+    (in_bom yes) (on_board no) (dnp no) (fields_autoplaced)
+    (property "Reference" "J4" (at 30.48 114.3 0)
+      (effects (font (size 1.27 1.27)))
+    )
+    (property "Value" "IDC20F" (at 30.48 116.84 0)
+      (effects (font (size 1.27 1.27)))
+    )
+    (property "Footprint" "" (at 30.48 142.24 0)
+      (effects (font (size 1.27 1.27)) hide)
+    )
+    (property "Datasheet" "~" (at 30.48 142.24 0)
+      (effects (font (size 1.27 1.27)) hide)
+    )
+    (pin "1")
+    (pin "10")
+    (pin "11")
+    (pin "12")
+    (pin "13")
+    (pin "14")
+    (pin "15")
+    (pin "16")
+    (pin "17")
+    (pin "18")
+    (pin "19")
+    (pin "2")
+    (pin "20")
+    (pin "3")
+    (pin "4")
+    (pin "5")
+    (pin "6")
+    (pin "7")
+    (pin "8")
+    (pin "9")
+    (instances
+      (project "SmartDiskII"
+        (path "/c5fa29fb-f00a-43d2-879f-1e361b003a2a"
+          (reference "J4") (unit 1)
+        )
+        (path "/c5fa29fb-f00a-43d2-879f-1e361b003a2a/4d4100c6-4979-4191-9309-82d4f93e23eb"
           (reference "J8") (unit 1)
         )
       )
-    )
-  )
-  (symbol (lib_id "Connector_Generic:Conn_01x20") (at 30.48 142.24 0) (mirror y) (unit 1)
-    (in_bom yes) (on_board no) (dnp no) (fields_autoplaced)
-    (property "Reference" "J4" (at 30.48 114.3 0)
-      (effects (font (size 1.27 1.27)))
-    )
-    (property "Value" "IDC20F" (at 30.48 116.84 0)
-      (effects (font (size 1.27 1.27)))
-    )
-    (property "Footprint" "" (at 30.48 142.24 0)
-      (effects (font (size 1.27 1.27)) hide)
-    )
-    (property "Datasheet" "~" (at 30.48 142.24 0)
-      (effects (font (size 1.27 1.27)) hide)
-    )
-    (pin "1")
-    (pin "10")
-    (pin "11")
-    (pin "12")
-    (pin "13")
-    (pin "14")
-    (pin "15")
-    (pin "16")
-    (pin "17")
-    (pin "18")
-    (pin "19")
-    (pin "2")
-    (pin "20")
-    (pin "3")
-    (pin "4")
-    (pin "5")
-    (pin "6")
-    (pin "7")
-    (pin "8")
-    (pin "9")
-    (instances
-      (project "SmartDiskII"
-        (path "/c5fa29fb-f00a-43d2-879f-1e361b003a2a"
-          (reference "J4") (unit 1)
-        )
-        (path "/c5fa29fb-f00a-43d2-879f-1e361b003a2a/4d4100c6-4979-4191-9309-82d4f93e23eb"
-          (reference "J7") (unit 1)
-        )
-      )

Commit message: Protect pin 12 with Diode
Connections:
- net SEL1 renamed SEL
Changed lines of the file:
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@@
     (effects (font (size 1.27 1.27)) (justify right bottom))
   )
-  (label "SEL1" (at 116.84 63.5 180) (fields_autoplaced)
+  (label "SEL" (at 116.84 63.5 180) (fields_autoplaced)
     (effects (font (size 1.27 1.27)) (justify right bottom))
   )
@@
     (effects (font (size 1.27 1.27)) (justify left bottom))
   )
-  (label "SEL1" (at 48.26 63.5 0) (fields_autoplaced)
+  (label "SEL" (at 48.26 63.5 0) (fields_autoplaced)
     (effects (font (size 1.27 1.27)) (justify left bottom))
   )
@@
     (effects (font (size 1.27 1.27)) (justify left bottom))
   )
-  (label "SEL1" (at 53.34 147.32 180) (fields_autoplaced)
+  (label "SEL" (at 53.34 147.32 180) (fields_autoplaced)
     (effects (font (size 1.27 1.27)) (justify right bottom))
   )
