File: SmartDiskII.kicad_sch (KiCad schematic)
At the start: 42 parts, among them J1 Apple II Expansion Slot, J2 DRV 1/SP, J3 DRV 2, U1 74LS174, U10 74LS30, U11 27C256, U12 74LS245, U13 74LS323, U14 74LS00, U2 NE556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

Commit message: housekeeping
Parts:
- JP1, JP2, JP3, JP4, JP5: now left out of the parts list
Changed lines of the file:
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@@
   )
   (symbol (lib_id "Jumper:SolderJumper_3_Bridged12") (at 200.66 154.94 90) (unit 1)
-    (in_bom yes) (on_board yes) (dnp no) (fields_autoplaced)
+    (in_bom no) (on_board yes) (dnp no) (fields_autoplaced)
     (property "Reference" "JP4" (at 198.12 154.305 90)
       (effects (font (size 1.27 1.27)) (justify left))
@@
   )
   (symbol (lib_id "Jumper:SolderJumper_2_Bridged") (at 313.69 27.94 0) (unit 1)
-    (in_bom yes) (on_board yes) (dnp no) (fields_autoplaced)
+    (in_bom no) (on_board yes) (dnp no) (fields_autoplaced)
     (property "Reference" "JP5" (at 313.69 24.13 0)
       (effects (font (size 1.27 1.27)))
@@
   )
   (symbol (lib_id "Jumper:SolderJumper_3_Bridged12") (at 295.91 25.4 90) (unit 1)
-    (in_bom yes) (on_board yes) (dnp no) (fields_autoplaced)
+    (in_bom no) (on_board yes) (dnp no) (fields_autoplaced)
     (property "Reference" "JP1" (at 293.37 26.035 90)
       (effects (font (size 1.27 1.27)) (justify left))
@@
   )
   (symbol (lib_id "Jumper:SolderJumper_2_Open") (at 311.15 40.64 0) (unit 1)
-    (in_bom yes) (on_board yes) (dnp no) (fields_autoplaced)
+    (in_bom no) (on_board yes) (dnp no) (fields_autoplaced)
     (property "Reference" "JP2" (at 311.15 38.1 0)
       (effects (font (size 1.27 1.27)))
@@
   )
   (symbol (lib_id "Jumper:SolderJumper_2_Open") (at 311.15 43.18 180) (unit 1)
-    (in_bom yes) (on_board yes) (dnp no) (fields_autoplaced)
+    (in_bom no) (on_board yes) (dnp no) (fields_autoplaced)
     (property "Reference" "JP3" (at 311.15 46.99 0)
       (effects (font (size 1.27 1.27)))
